File: sdi.kicad_sch (KiCad schematic)
At the start: 50 parts, among them J2 031-70526-21, J3 031-70526-21, U11 LIFCL-40-9BG256C, U15 GS2971A, U16 GS2988, Y1 ABM7_27.000MH_D2Y_T

Commit message: Placed components
Parts:
- C40: renamed from C58; value C_100n_0603 -> C_100n_0402; footprint crosslink-nx-video-converter-footprints:0603-cap -> antmicro-footprints:0402-cap; symbol crosslink-nx-video-converter:C_100n_0603 -> antmicroCapacitors0402:C_100n_0402; MPN 0603YC104KAZ2A -> GRM155R61H104KE14D; Manufacturer AVX -> Murata
- C51, C52: value C_33p_0603 -> C_33p_0402; footprint crosslink-nx-video-converter-footprints:0603-cap -> antmicro-footprints:0402-cap; symbol crosslink-nx-video-converter:C_33p_0603 -> antmicroCapacitors0402:C_33p_0402; MPN 06031A330JAT2A -> MC0402N330J500CT; Manufacturer AVX -> MULTICOMP
- C58: renamed from C60; value C_100n_0603 -> C_100n_0402; footprint crosslink-nx-video-converter-footprints:0603-cap -> antmicro-footprints:0402-cap; symbol crosslink-nx-video-converter:C_100n_0603 -> antmicroCapacitors0402:C_100n_0402; MPN 0603YC104KAZ2A -> GRM155R61H104KE14D; Manufacturer AVX -> Murata
- C60: renamed from C61; value C_100n_0603 -> C_100n_0402; footprint crosslink-nx-video-converter-footprints:0603-cap -> antmicro-footprints:0402-cap; symbol crosslink-nx-video-converter:C_100n_0603 -> antmicroCapacitors0402:C_100n_0402; MPN 0603YC104KAZ2A -> GRM155R61H104KE14D; Manufacturer AVX -> Murata
- C61: renamed from C62; value C_100n_0603 -> C_100n_0402; footprint crosslink-nx-video-converter-footprints:0603-cap -> antmicro-footprints:0402-cap; symbol crosslink-nx-video-converter:C_100n_0603 -> antmicroCapacitors0402:C_100n_0402; MPN 0603YC104KAZ2A -> GRM155R61H104KE14D; Manufacturer AVX -> Murata
- C62: renamed from C63; value C_100n_0603 -> C_100n_0402; footprint crosslink-nx-video-converter-footprints:0603-cap -> antmicro-footprints:0402-cap; symbol crosslink-nx-video-converter:C_100n_0603 -> antmicroCapacitors0402:C_100n_0402; MPN 0603YC104KAZ2A -> GRM155R61H104KE14D; Manufacturer AVX -> Murata
- C63: renamed from C64; value C_100n_0603 -> C_100n_0402; footprint crosslink-nx-video-converter-footprints:0603-cap -> antmicro-footprints:0402-cap; symbol crosslink-nx-video-converter:C_100n_0603 -> antmicroCapacitors0402:C_100n_0402; MPN 0603YC104KAZ2A -> GRM155R61H104KE14D; Manufacturer AVX -> Murata
- C64: renamed from C65; value C_100n_0603 -> C_100n_0402; footprint crosslink-nx-video-converter-footprints:0603-cap -> antmicro-footprints:0402-cap; symbol crosslink-nx-video-converter:C_100n_0603 -> antmicroCapacitors0402:C_100n_0402; MPN 0603YC104KAZ2A -> GRM155R61H104KE14D; Manufacturer AVX -> Murata
- C65: renamed from C66; value C_100n_0603 -> C_100n_0402; footprint crosslink-nx-video-converter-footprints:0603-cap -> antmicro-footprints:0402-cap; symbol crosslink-nx-video-converter:C_100n_0603 -> antmicroCapacitors0402:C_100n_0402; MPN 0603YC104KAZ2A -> GRM155R61H104KE14D; Manufacturer AVX -> Murata
- C66: renamed from C67; value C_100n_0603 -> C_100n_0402; footprint crosslink-nx-video-converter-footprints:0603-cap -> antmicro-footprints:0402-cap; symbol crosslink-nx-video-converter:C_100n_0603 -> antmicroCapacitors0402:C_100n_0402; MPN 0603YC104KAZ2A -> GRM155R61H104KE14D; Manufacturer AVX -> Murata
- C67: renamed from C68; value C_100n_0603 -> C_100n_0402; footprint crosslink-nx-video-converter-footprints:0603-cap -> antmicro-footprints:0402-cap; symbol crosslink-nx-video-converter:C_100n_0603 -> antmicroCapacitors0402:C_100n_0402; MPN 0603YC104KAZ2A -> GRM155R61H104KE14D; Manufacturer AVX -> Murata
- C68: renamed from C69; value C_100n_0603 -> C_100n_0402; footprint crosslink-nx-video-converter-footprints:0603-cap -> antmicro-footprints:0402-cap; symbol crosslink-nx-video-converter:C_100n_0603 -> antmicroCapacitors0402:C_100n_0402; MPN 0603YC104KAZ2A -> GRM155R61H104KE14D; Manufacturer AVX -> Murata
- C69: renamed from C70; value C_100n_0603 -> C_100n_0402; footprint crosslink-nx-video-converter-footprints:0603-cap -> antmicro-footprints:0402-cap; symbol crosslink-nx-video-converter:C_100n_0603 -> antmicroCapacitors0402:C_100n_0402; MPN 0603YC104KAZ2A -> GRM155R61H104KE14D; Manufacturer AVX -> Murata
- C70: renamed from C72; value C_100n_0603 -> C_100n_0402; footprint crosslink-nx-video-converter-footprints:0603-cap -> antmicro-footprints:0402-cap; symbol crosslink-nx-video-converter:C_100n_0603 -> antmicroCapacitors0402:C_100n_0402; MPN 0603YC104KAZ2A -> GRM155R61H104KE14D; Manufacturer AVX -> Murata
- C72: renamed from C73; value C_100n_0603 -> C_100n_0402; footprint crosslink-nx-video-converter-footprints:0603-cap -> antmicro-footprints:0402-cap; symbol crosslink-nx-video-converter:C_100n_0603 -> antmicroCapacitors0402:C_100n_0402; MPN 0603YC104KAZ2A -> GRM155R61H104KE14D; Manufacturer AVX -> Murata
- C73: renamed from C74; value C_100n_0603 -> C_100n_0402; footprint crosslink-nx-video-converter-footprints:0603-cap -> antmicro-footprints:0402-cap; symbol crosslink-nx-video-converter:C_100n_0603 -> antmicroCapacitors0402:C_100n_0402; MPN 0603YC104KAZ2A -> GRM155R61H104KE14D; Manufacturer AVX -> Murata
- C74: renamed from C75; value C_100n_0603 -> C_100n_0402; footprint crosslink-nx-video-converter-footprints:0603-cap -> antmicro-footprints:0402-cap; symbol crosslink-nx-video-converter:C_100n_0603 -> antmicroCapacitors0402:C_100n_0402; MPN 0603YC104KAZ2A -> GRM155R61H104KE14D; Manufacturer AVX -> Murata
- R38: renamed from R58; value R_0R_0603 -> R_0R_0402; footprint crosslink-nx-video-converter-footprints:0603-res -> antmicro-footprints:0402-res; symbol crosslink-nx-video-converter:R_0R_0603 -> antmicroResistors0402:R_0R_0402; MPN CR0603-J/-000ELF -> ERJ2GE0R00X; Manufacturer BOURNS -> PANASONIC
- R54, R55: value R_100k_0603 -> R_100k_0402; footprint crosslink-nx-video-converter-footprints:0603-res -> antmicro-footprints:0402-res; symbol crosslink-nx-video-converter:R_100k_0603 -> antmicroResistors0402:R_100k_0402; DNP DNP -> (none); MPN CR0603-FX-1003HLF -> CRCW0402100KFKEDHP; Manufacturer BOURNS -> VISHAY
- TP13: renamed from TP14; value TP -> TP_SMD_0_75MM; footprint crosslink-nx-video-converter-footprints:TP-R-1.5 -> antmicro-footprints:Testpoint_smd_0_75mm; symbol crosslink-nx-video-converter:TP -> antmicroTestPoints:TP_SMD_0_75MM
- TP14: renamed from TP15; value TP -> TP_SMD_0_75MM; footprint crosslink-nx-video-converter-footprints:TP-R-1.5 -> antmicro-footprints:Testpoint_smd_0_75mm; symbol crosslink-nx-video-converter:TP -> antmicroTestPoints:TP_SMD_0_75MM
