File: crosslink-nx-video-converter.kicad_sch (KiCad schematic)
At the start: 0 parts

Commit message: Added revision and title to the schematic sheets
Other:
- title: (none) -> CrossLink-NX Video Converter
Changed lines of the file:
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@@
 (kicad_sch (version 20211123) (generator eeschema)
   (paper "A3")
+  (title_block
+    (title "CrossLink-NX Video Converter")
+    (date "2022-10-27")
+    (rev "1.0.0")
+    (comment 1 "www.antmicro.com")
+    (comment 2 "Antmicro Ltd.")
+  )
   (image (at 208.28 127) (scale 1.36675)
     (data
