File: supply.kicad_sch (KiCad schematic)
At the start: 107 parts, among them Q1 2N7002, Q2 BCM857BS-7-F, Q3 AO3401A, U1 MP20073, U10 AP7330-W5-7, U2 LM339, U3 LM339, U4 DIO7553ST6, U5 AP62301WU-7, U6 AP62301WU-7, U7 AP62301WU-7, U8 AP7330-W5-7, U9 AP7330-W5-7

Commit message: Update project naming convention
Parts:
- C1, C14, C15, C2, C3, C6, C9: footprint crosslink-nx-video-converter-footprints:0402-cap -> sdi-mipi-cross-converter-footprints:0402-cap; symbol crosslink-nx-video-converter:C_100n_0402 -> sdi-mipi-cross-converter:C_100n_0402
- C10, C108, C11, C12, C13, C31: footprint crosslink-nx-video-converter-footprints:0603-cap -> sdi-mipi-cross-converter-footprints:0603-cap; symbol crosslink-nx-video-converter:C_10u_0603 -> sdi-mipi-cross-converter:C_10u_0603
- C17, C18, C19, C29, C30, C4: footprint crosslink-nx-video-converter-footprints:0603-cap -> sdi-mipi-cross-converter-footprints:0603-cap; symbol crosslink-nx-video-converter:C_1u_0603 -> sdi-mipi-cross-converter:C_1u_0603
- C20, C21, C22, C23, C24, C25, C26, C27, C28, C32, C33, C34, C5, C7, C8: footprint crosslink-nx-video-converter-footprints:0603-cap -> sdi-mipi-cross-converter-footprints:0603-cap; symbol crosslink-nx-video-converter:C_22u_0603 -> sdi-mipi-cross-converter:C_22u_0603
- D1, D2: footprint crosslink-nx-video-converter-footprints:LED_0603 -> sdi-mipi-cross-converter-footprints:LED_0603; symbol crosslink-nx-video-converter:LTST-C190GKT -> sdi-mipi-cross-converter:LTST-C190GKT
- L1, L2, L3: footprint crosslink-nx-video-converter-footprints:Coilcraft-XEL4030 -> sdi-mipi-cross-converter-footprints:Coilcraft-XEL4030; symbol crosslink-nx-video-converter:XEL4030-332MEC -> sdi-mipi-cross-converter:XEL4030-332MEC
- Q1: footprint crosslink-nx-video-converter-footprints:SOT-23-3 -> sdi-mipi-cross-converter-footprints:SOT-23-3; symbol crosslink-nx-video-converter:2N7002 -> sdi-mipi-cross-converter:2N7002
- Q2: footprint crosslink-nx-video-converter-footprints:SOT-363 -> sdi-mipi-cross-converter-footprints:SOT-363; symbol crosslink-nx-video-converter:BCM857BS-7-F -> sdi-mipi-cross-converter:BCM857BS-7-F
- Q3: footprint crosslink-nx-video-converter-footprints:SOT-23-3 -> sdi-mipi-cross-converter-footprints:SOT-23-3; symbol crosslink-nx-video-converter:AO3401A -> sdi-mipi-cross-converter:AO3401A
- R1: footprint crosslink-nx-video-converter-footprints:0402-res -> sdi-mipi-cross-converter-footprints:0402-res; symbol crosslink-nx-video-converter:R_100k_0402 -> sdi-mipi-cross-converter:R_100k_0402
- R10: footprint crosslink-nx-video-converter-footprints:0402-res -> sdi-mipi-cross-converter-footprints:0402-res; symbol crosslink-nx-video-converter:R_1k3_0402 -> sdi-mipi-cross-converter:R_1k3_0402
- R12: footprint crosslink-nx-video-converter-footprints:0402-res -> sdi-mipi-cross-converter-footprints:0402-res; symbol crosslink-nx-video-converter:R_1k5_0402 -> sdi-mipi-cross-converter:R_1k5_0402
- R13, R4: footprint crosslink-nx-video-converter-footprints:1206-res -> sdi-mipi-cross-converter-footprints:1206-res; symbol crosslink-nx-video-converter:R_0R_1206 -> sdi-mipi-cross-converter:R_0R_1206
- R14, R18: footprint crosslink-nx-video-converter-footprints:0402-res -> sdi-mipi-cross-converter-footprints:0402-res; symbol crosslink-nx-video-converter:R_470R_0402 -> sdi-mipi-cross-converter:R_470R_0402
- R15, R16, R17, R40, R41, R42, R5: footprint crosslink-nx-video-converter-footprints:0805-res -> sdi-mipi-cross-converter-footprints:0805-res; symbol crosslink-nx-video-converter:R_0R_0805 -> sdi-mipi-cross-converter:R_0R_0805
- R19, R20, R21, R24, R25, R28: footprint crosslink-nx-video-converter-footprints:0402-res -> sdi-mipi-cross-converter-footprints:0402-res; symbol crosslink-nx-video-converter:R_0R_0402 -> sdi-mipi-cross-converter:R_0R_0402
- R2, R23, R27, R32, R6, R63, R64, R9, R98, R99: footprint crosslink-nx-video-converter-footprints:0402-res -> sdi-mipi-cross-converter-footprints:0402-res; symbol crosslink-nx-video-converter:R_10k_0402 -> sdi-mipi-cross-converter:R_10k_0402
- R22, R31: footprint crosslink-nx-video-converter-footprints:0402-res -> sdi-mipi-cross-converter-footprints:0402-res; symbol crosslink-nx-video-converter:R_3k01_0402 -> sdi-mipi-cross-converter:R_3k01_0402
- R26: footprint crosslink-nx-video-converter-footprints:0402-res -> sdi-mipi-cross-converter-footprints:0402-res; symbol crosslink-nx-video-converter:R_33k_0402 -> sdi-mipi-cross-converter:R_33k_0402
- R29, R30, R37: footprint crosslink-nx-video-converter-footprints:0603-res -> sdi-mipi-cross-converter-footprints:0603-res; symbol crosslink-nx-video-converter:R_0R_0603 -> sdi-mipi-cross-converter:R_0R_0603
- R3: footprint crosslink-nx-video-converter-footprints:0402-res -> sdi-mipi-cross-converter-footprints:0402-res; symbol crosslink-nx-video-converter:R_1k_0402 -> sdi-mipi-cross-converter:R_1k_0402
- R33: footprint crosslink-nx-video-converter-footprints:0402-res -> sdi-mipi-cross-converter-footprints:0402-res; symbol crosslink-nx-video-converter:R_12k_0402 -> sdi-mipi-cross-converter:R_12k_0402
- R34: footprint crosslink-nx-video-converter-footprints:0402-res -> sdi-mipi-cross-converter-footprints:0402-res; symbol crosslink-nx-video-converter:R_24k_0402 -> sdi-mipi-cross-converter:R_24k_0402
- R35: footprint crosslink-nx-video-converter-footprints:0402-res -> sdi-mipi-cross-converter-footprints:0402-res; symbol crosslink-nx-video-converter:R_18k7_0402 -> sdi-mipi-cross-converter:R_18k7_0402
- R36: footprint crosslink-nx-video-converter-footprints:0402-res -> sdi-mipi-cross-converter-footprints:0402-res; symbol crosslink-nx-video-converter:R_15k_0402 -> sdi-mipi-cross-converter:R_15k_0402
- R7: footprint crosslink-nx-video-converter-footprints:0402-res -> sdi-mipi-cross-converter-footprints:0402-res; symbol crosslink-nx-video-converter:R_22R_0402 -> sdi-mipi-cross-converter:R_22R_0402
- TP1, TP10, TP11, TP12, TP2, TP23, TP3, TP4, TP5, TP6, TP7, TP8, TP9: footprint crosslink-nx-video-converter-footprints:Testpoint_smd_0_75mm -> sdi-mipi-cross-converter-footprints:Testpoint_smd_0_75mm; symbol crosslink-nx-video-converter:TP_SMD_0_75MM -> sdi-mipi-cross-converter:TP_SMD_0_75MM
- U1: footprint crosslink-nx-video-converter-footprints:MSOP-8-1EP_W3mm -> sdi-mipi-cross-converter-footprints:MSOP-8-1EP_W3mm; symbol crosslink-nx-video-converter:MP20073 -> sdi-mipi-cross-converter:MP20073
- U10, U8, U9: footprint crosslink-nx-video-converter-footprints:SOT-23-5 -> sdi-mipi-cross-converter-footprints:SOT-23-5; symbol crosslink-nx-video-converter:AP7330-W5-7 -> sdi-mipi-cross-converter:AP7330-W5-7
- U2, U3: footprint crosslink-nx-video-converter-footprints:TSSOP-14_4.4x5mm_P0.65mm -> sdi-mipi-cross-converter-footprints:TSSOP-14_4.4x5mm_P0.65mm; symbol crosslink-nx-video-converter: LM339 -> sdi-mipi-cross-converter: LM339
- U4: footprint crosslink-nx-video-converter-footprints:SOT23-6L -> sdi-mipi-cross-converter-footprints:SOT23-6L; symbol crosslink-nx-video-converter:DIO7553ST6 -> sdi-mipi-cross-converter:DIO7553ST6
- U5, U6, U7: footprint crosslink-nx-video-converter-footprints:TSOT23-6 -> sdi-mipi-cross-converter-footprints:TSOT23-6; symbol crosslink-nx-video-converter:AP62301WU-7 -> sdi-mipi-cross-converter:AP62301WU-7

Commit message: Bump to 1.1.0, update naming
Other:
- title: CrossLink-NX Video Converter -> SDI-MIPI Cross Converter
