File: sdi-mipi-cross-converter.kicad_sch (KiCad schematic)
At the start: 0 parts

Commit message: Bump to 1.1.0, update naming
Other:
- title: CrossLink-NX Video Converter -> SDI-MIPI Cross Converter
