File: peripherals.kicad_sch (KiCad schematic)
At the start: 75 parts, among them J1 USB4105-GF-A, J10 TSM-106-01-T-SH, J4 WE_68715014522_ONE-SIDE, J5 FTSH-105-01-F-DV-K, J6 WE_68715014522_ONE-SIDE, J8 SM04B-SRSS-TB-LF-SN, J9 SM06B-SRSS-TB(LF)(SN), SW1 CVS-02B, U11 LIFCL-40-9BG256C, U13 DIO7553ST6, U14 DIO7553ST6, U19 DIO7553ST6, U20 FT230XQ-R

Commit message: Added revision and title to the schematic sheets
Other:
- title: (none) -> CrossLink-NX Video Converter
Changed lines of the file:
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@@
 (kicad_sch (version 20211123) (generator eeschema)
   (paper "A3")
+  (title_block
+    (title "CrossLink-NX Video Converter")
+    (date "2022-10-27")
+    (rev "1.0.0")
+    (comment 1 "www.antmicro.com")
+    (comment 2 "Antmicro Ltd.")
+  )
   (junction (at 157.48 214.63) (diameter 0) (color 0 0 0 0)
   )

Commit message: Update PCB routing
- apply new DRC
- add FPGA package delay to the high speed traces tunning
- improve GND and power planes
Parts:
- removed C83, C84: C_100n_0402, crosslink-nx-video-converter-footprints:0402-cap, symbol crosslink-nx-video-converter:C_100n_0402
- added C83, C84: C_100n_0201, crosslink-nx-video-converter-footprints:0201-res, symbol crosslink-nx-video-converter:C_100n_0201
- U11: footprint crosslink-nx-video-converter-footprints:BGA-256_16x16_14.0x14.0mm -> crosslink-nx-video-converter-footprints:CrosslinkNX-BGA-256_16x16_14.0x14.0mm
Connections:
- net +1V2: now also C83.1
- net +3V3: now also C84.1
- net DIP0: now also U11.F15 (PR13B)
- net FCC2_SCL2: no longer U11.F15 (PR13B)
- net FFC1_3V3: now also J4.47 (Pin_47), J4.48 (Pin_48)
- net FFC1_5V: now also J4.49 (Pin_49), J4.50 (Pin_50)
- net GND: now also J4.12 (Pin_12), J4.15 (Pin_15), J4.18 (Pin_18), J4.27 (Pin_27), J4.30 (Pin_30), J4.9 (Pin_9), J4.SH (SHLD), C83.2, C84.2
- net MIPI0_CLK_N: now also J4.10 (Pin_10)
- net MIPI0_CLK_P: now also J4.11 (Pin_11)
- net MIPI0_D0_N: now also J4.7 (Pin_7)
- net MIPI0_D0_P: now also J4.8 (Pin_8)
- net MIPI0_D1_N: now also J4.5 (Pin_5)
- net MIPI0_D1_P: now also J4.6 (Pin_6)
- net MIPI0_D2_N: now also J4.3 (Pin_3)
- net MIPI0_D2_P: now also J4.4 (Pin_4)
- net MIPI0_D3_N: now also J4.1 (Pin_1)
- net MIPI0_D3_P: now also J4.2 (Pin_2)
- net MIPI2_CLK_N: now also J4.28 (Pin_28)
- net MIPI2_CLK_P: now also J4.29 (Pin_29)
- net MIPI2_D0_N: now also J4.25 (Pin_25)
- net MIPI2_D0_P: now also J4.26 (Pin_26)
- net MIPI2_D1_N: now also J4.23 (Pin_23)
- net MIPI2_D1_P: now also J4.24 (Pin_24)
- net MIPI2_D2_N: now also J4.21 (Pin_21)
- net MIPI2_D2_P: now also J4.22 (Pin_22)
- net MIPI2_D3_N: now also J4.19 (Pin_19)
- net MIPI2_D3_P: now also J4.20 (Pin_20)
- net at R122.2: now also J4.39 (Pin_39)
- net at R124.2: now also J4.41 (Pin_41)
- net at R121.2: now also J4.34 (Pin_34)
- net at R74.2: now also J4.33 (Pin_33)
- net at R123.1: now also J4.40 (Pin_40)
- net at R125.1: now also J4.42 (Pin_42)
- net at R73.2: now also J4.32 (Pin_32)

Commit message: Update project naming convention
Parts:
- C109, C110, C113, C122, C123: footprint crosslink-nx-video-converter-footprints:0402-cap -> sdi-mipi-cross-converter-footprints:0402-cap; symbol crosslink-nx-video-converter:C_100n_0402 -> sdi-mipi-cross-converter:C_100n_0402
- C111, C112, C114, C124: footprint crosslink-nx-video-converter-footprints:0603-cap -> sdi-mipi-cross-converter-footprints:0603-cap; symbol crosslink-nx-video-converter:C_1u_0603 -> sdi-mipi-cross-converter:C_1u_0603
- C117, C121: footprint crosslink-nx-video-converter-footprints:0402-cap -> sdi-mipi-cross-converter-footprints:0402-cap; symbol crosslink-nx-video-converter:C_47p_0402 -> sdi-mipi-cross-converter:C_47p_0402
- C83, C84: footprint crosslink-nx-video-converter-footprints:0201-res -> sdi-mipi-cross-converter-footprints:0201-res; symbol crosslink-nx-video-converter:C_100n_0201 -> sdi-mipi-cross-converter:C_100n_0201
- D10, D11, D12, D13, D3, D4, D9: footprint crosslink-nx-video-converter-footprints:LED_0603 -> sdi-mipi-cross-converter-footprints:LED_0603; symbol crosslink-nx-video-converter:LTST-C190GKT -> sdi-mipi-cross-converter:LTST-C190GKT
- F1: footprint crosslink-nx-video-converter-footprints:0603-Fuse-Littelfuse-0467 -> sdi-mipi-cross-converter-footprints:0603-Fuse-Littelfuse-0467; symbol crosslink-nx-video-converter:04671.25NR -> sdi-mipi-cross-converter:04671.25NR
- J1: footprint crosslink-nx-video-converter-footprints:GCT_USB4105-GF-A -> sdi-mipi-cross-converter-footprints:GCT_USB4105-GF-A; symbol crosslink-nx-video-converter:USB4105-GF-A -> sdi-mipi-cross-converter:USB4105-GF-A
- J10: footprint crosslink-nx-video-converter-footprints:SAMTEC_TSM-106-01-T-SH -> sdi-mipi-cross-converter-footprints:SAMTEC_TSM-106-01-T-SH; symbol crosslink-nx-video-converter:TSM-106-01-T-SH -> sdi-mipi-cross-converter:TSM-106-01-T-SH
- J4, J6: footprint crosslink-nx-video-converter-footprints:WE_68715014522_ONE-SIDE -> sdi-mipi-cross-converter-footprints:WE_68715014522_ONE-SIDE; symbol crosslink-nx-video-converter:WE_68715014522_ONE-SIDE -> sdi-mipi-cross-converter:WE_68715014522_ONE-SIDE
- J5: footprint crosslink-nx-video-converter-footprints:PinHeader_2x5_P1.27_SMD -> sdi-mipi-cross-converter-footprints:PinHeader_2x5_P1.27_SMD; symbol crosslink-nx-video-converter:FTSH-105-01-F-DV-K -> sdi-mipi-cross-converter:FTSH-105-01-F-DV-K
- J8: footprint crosslink-nx-video-converter-footprints:SM04B-SRSS-TB-LF-SN -> sdi-mipi-cross-converter-footprints:SM04B-SRSS-TB-LF-SN; symbol crosslink-nx-video-converter:SM04B-SRSS-TB-LF-SN -> sdi-mipi-cross-converter:SM04B-SRSS-TB-LF-SN
- J9: footprint crosslink-nx-video-converter-footprints:JST_SM06B-SRSS-TB(LF)(SN) -> sdi-mipi-cross-converter-footprints:JST_SM06B-SRSS-TB(LF)(SN); symbol crosslink-nx-video-converter:SM06B-SRSS-TB(LF)(SN) -> sdi-mipi-cross-converter:SM06B-SRSS-TB(LF)(SN)
- R102, R111, R112, R120, R135, R136: footprint crosslink-nx-video-converter-footprints:0603-res -> sdi-mipi-cross-converter-footprints:0603-res; symbol crosslink-nx-video-converter:R_200R_0603 -> sdi-mipi-cross-converter:R_200R_0603
- R103: footprint crosslink-nx-video-converter-footprints:0603-res -> sdi-mipi-cross-converter-footprints:0603-res; symbol crosslink-nx-video-converter:R_470R_0603 -> sdi-mipi-cross-converter:R_470R_0603
- R104, R105, R106, R113, R114, R115: footprint crosslink-nx-video-converter-footprints:0603-res -> sdi-mipi-cross-converter-footprints:0603-res; symbol crosslink-nx-video-converter:R_10k_0603 -> sdi-mipi-cross-converter:R_10k_0603
- R107, R108, R118: footprint crosslink-nx-video-converter-footprints:0603-res -> sdi-mipi-cross-converter-footprints:0603-res; symbol crosslink-nx-video-converter:R_15k_0603 -> sdi-mipi-cross-converter:R_15k_0603
- R109, R110, R121, R122, R123, R124, R125, R126, R127, R128, R129, R130, R73, R74: footprint crosslink-nx-video-converter-footprints:0402-res -> sdi-mipi-cross-converter-footprints:0402-res; symbol crosslink-nx-video-converter:R_0R_0402 -> sdi-mipi-cross-converter:R_0R_0402
- R11, R8: footprint crosslink-nx-video-converter-footprints:0402-res -> sdi-mipi-cross-converter-footprints:0402-res; symbol crosslink-nx-video-converter:R_5k1_0402 -> sdi-mipi-cross-converter:R_5k1_0402
- R116, R117, R119: footprint crosslink-nx-video-converter-footprints:0603-res -> sdi-mipi-cross-converter-footprints:0603-res; symbol crosslink-nx-video-converter:R_0R_0603 -> sdi-mipi-cross-converter:R_0R_0603
- R133, R134: footprint crosslink-nx-video-converter-footprints:0402-res -> sdi-mipi-cross-converter-footprints:0402-res; symbol crosslink-nx-video-converter:R_27R_0402 -> sdi-mipi-cross-converter:R_27R_0402
- SW1: footprint crosslink-nx-video-converter-footprints:SW_DIP_SPSTx02_Slide_Copal_CVS-02xB_W5.9mm_P1mm -> sdi-mipi-cross-converter-footprints:SW_DIP_SPSTx02_Slide_Copal_CVS-02xB_W5.9mm_P1mm; symbol crosslink-nx-video-converter:CVS-02B -> sdi-mipi-cross-converter:CVS-02B
- TP44, TP45, TP46, TP47: footprint crosslink-nx-video-converter-footprints:Testpoint_smd_0_75mm -> sdi-mipi-cross-converter-footprints:Testpoint_smd_0_75mm; symbol crosslink-nx-video-converter:TP_SMD_0_75MM -> sdi-mipi-cross-converter:TP_SMD_0_75MM
- U11: footprint crosslink-nx-video-converter-footprints:CrosslinkNX-BGA-256_16x16_14.0x14.0mm -> sdi-mipi-cross-converter-footprints:CrosslinkNX-BGA-256_16x16_14.0x14.0mm; symbol crosslink-nx-video-converter:LIFCL-40-9BG256C -> sdi-mipi-cross-converter:LIFCL-40-9BG256C
- U13, U14, U19: footprint crosslink-nx-video-converter-footprints:SOT23-6L -> sdi-mipi-cross-converter-footprints:SOT23-6L; symbol crosslink-nx-video-converter:DIO7553ST6 -> sdi-mipi-cross-converter:DIO7553ST6
- U20: footprint crosslink-nx-video-converter-footprints:WQFN-16-1EP_4x4mm -> sdi-mipi-cross-converter-footprints:WQFN-16-1EP_4x4mm; symbol crosslink-nx-video-converter:FT230XQ-R -> sdi-mipi-cross-converter:FT230XQ-R

Commit message: Bump to 1.1.0, update naming
Other:
- title: CrossLink-NX Video Converter -> SDI-MIPI Cross Converter

Commit message: Update U11/LIFCL-40-9BG256C footprint property
Parts:
- U11: footprint sdi-mipi-cross-converter-footprints:CrosslinkNX-BGA-256_16x16_14.0x14.0mm -> sdi-mipi-cross-converter-footprints:BGA-256_16x16_14.0x14.0mm
Changed lines of the file:
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@@
     (property "Reference" "U11" (id 0) (at 64.77 72.39 0))
     (property "Value" "LIFCL-40-9BG256C" (id 1) (at 64.77 74.93 0))
-    (property "Footprint" "sdi-mipi-cross-converter-footprints:CrosslinkNX-BGA-256_16x16_14.0x14.0mm" (id 2) (at 66.675 235.585 0)
+    (property "Footprint" "sdi-mipi-cross-converter-footprints:BGA-256_16x16_14.0x14.0mm" (id 2) (at 66.675 235.585 0)
       (effects (font (size 1.27 1.27)) hide)
     )
@@
     (property "Reference" "U11" (id 0) (at 37.465 25.4 0))
     (property "Value" "LIFCL-40-9BG256C" (id 1) (at 37.465 27.94 0))
-    (property "Footprint" "sdi-mipi-cross-converter-footprints:CrosslinkNX-BGA-256_16x16_14.0x14.0mm" (id 2) (at 40.005 187.325 0)
+    (property "Footprint" "sdi-mipi-cross-converter-footprints:BGA-256_16x16_14.0x14.0mm" (id 2) (at 40.005 187.325 0)
       (effects (font (size 1.27 1.27)) hide)
     )
@@
     (property "Reference" "U11" (id 0) (at 92.075 25.4 0))
     (property "Value" "LIFCL-40-9BG256C" (id 1) (at 92.075 27.94 0))
-    (property "Footprint" "sdi-mipi-cross-converter-footprints:CrosslinkNX-BGA-256_16x16_14.0x14.0mm" (id 2) (at 93.345 187.325 0)
+    (property "Footprint" "sdi-mipi-cross-converter-footprints:BGA-256_16x16_14.0x14.0mm" (id 2) (at 93.345 187.325 0)
       (effects (font (size 1.27 1.27)) hide)
     )
@@
     (property "Reference" "U11" (id 0) (at 55.88 118.11 0))
     (property "Value" "LIFCL-40-9BG256C" (id 1) (at 55.88 120.65 0))
-    (property "Footprint" "sdi-mipi-cross-converter-footprints:CrosslinkNX-BGA-256_16x16_14.0x14.0mm" (id 2) (at 57.785 294.005 0)
-      (effects (font (size 1.27 1.27)) hide)
-    )
+    (property "Footprint" "sdi-mipi-cross-converter-footprints:BGA-256_16x16_14.0x14.0mm" (id 2) (at 57.785 294.005 0)
+      (effects (font (size 1.27 1.27)) hide)
+    )

Commit message: Add logotypes to schematics
Other:
- moved on the sheet: C113, C114, D11, J8, R113, R114, R115, R116, R117, R118, R120, TP45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

Commit message: Update naming convention
Parts:
- C109, C110, C113, C122, C123: footprint sdi-mipi-cross-converter-footprints:0402-cap -> sdi-mipi-video-converter-footprints:0402-cap; symbol sdi-mipi-cross-converter:C_100n_0402 -> sdi-mipi-video-converter:C_100n_0402
- C111, C112, C114, C124: footprint sdi-mipi-cross-converter-footprints:0603-cap -> sdi-mipi-video-converter-footprints:0603-cap; symbol sdi-mipi-cross-converter:C_1u_0603 -> sdi-mipi-video-converter:C_1u_0603
- C117, C121: footprint sdi-mipi-cross-converter-footprints:0402-cap -> sdi-mipi-video-converter-footprints:0402-cap; symbol sdi-mipi-cross-converter:C_47p_0402 -> sdi-mipi-video-converter:C_47p_0402
- C83, C84: footprint sdi-mipi-cross-converter-footprints:0201-res -> sdi-mipi-video-converter-footprints:0201-res; symbol sdi-mipi-cross-converter:C_100n_0201 -> sdi-mipi-video-converter:C_100n_0201
- D10, D11, D12, D13, D3, D4, D9: footprint sdi-mipi-cross-converter-footprints:LED_0603 -> sdi-mipi-video-converter-footprints:LED_0603; symbol sdi-mipi-cross-converter:LTST-C190GKT -> sdi-mipi-video-converter:LTST-C190GKT
- F1: footprint sdi-mipi-cross-converter-footprints:0603-Fuse-Littelfuse-0467 -> sdi-mipi-video-converter-footprints:0603-Fuse-Littelfuse-0467; symbol sdi-mipi-cross-converter:04671.25NR -> sdi-mipi-video-converter:04671.25NR
- J1: footprint sdi-mipi-cross-converter-footprints:GCT_USB4105-GF-A -> sdi-mipi-video-converter-footprints:GCT_USB4105-GF-A; symbol sdi-mipi-cross-converter:USB4105-GF-A -> sdi-mipi-video-converter:USB4105-GF-A
- J10: footprint sdi-mipi-cross-converter-footprints:SAMTEC_TSM-106-01-T-SH -> sdi-mipi-video-converter-footprints:SAMTEC_TSM-106-01-T-SH; symbol sdi-mipi-cross-converter:TSM-106-01-T-SH -> sdi-mipi-video-converter:TSM-106-01-T-SH
- J4, J6: footprint sdi-mipi-cross-converter-footprints:WE_68715014522_ONE-SIDE -> sdi-mipi-video-converter-footprints:WE_68715014522_ONE-SIDE; symbol sdi-mipi-cross-converter:WE_68715014522_ONE-SIDE -> sdi-mipi-video-converter:WE_68715014522_ONE-SIDE
- J5: footprint sdi-mipi-cross-converter-footprints:PinHeader_2x5_P1.27_SMD -> sdi-mipi-video-converter-footprints:PinHeader_2x5_P1.27_SMD; symbol sdi-mipi-cross-converter:FTSH-105-01-F-DV-K -> sdi-mipi-video-converter:FTSH-105-01-F-DV-K
- J8: footprint sdi-mipi-cross-converter-footprints:SM04B-SRSS-TB-LF-SN -> sdi-mipi-video-converter-footprints:SM04B-SRSS-TB-LF-SN; symbol sdi-mipi-cross-converter:SM04B-SRSS-TB-LF-SN -> sdi-mipi-video-converter:SM04B-SRSS-TB-LF-SN
- J9: footprint sdi-mipi-cross-converter-footprints:JST_SM06B-SRSS-TB(LF)(SN) -> sdi-mipi-video-converter-footprints:JST_SM06B-SRSS-TB(LF)(SN); symbol sdi-mipi-cross-converter:SM06B-SRSS-TB(LF)(SN) -> sdi-mipi-video-converter:SM06B-SRSS-TB(LF)(SN)
- R102, R111, R112, R120, R135, R136: footprint sdi-mipi-cross-converter-footprints:0603-res -> sdi-mipi-video-converter-footprints:0603-res; symbol sdi-mipi-cross-converter:R_200R_0603 -> sdi-mipi-video-converter:R_200R_0603
- R103: footprint sdi-mipi-cross-converter-footprints:0603-res -> sdi-mipi-video-converter-footprints:0603-res; symbol sdi-mipi-cross-converter:R_470R_0603 -> sdi-mipi-video-converter:R_470R_0603
- R104, R105, R106, R113, R114, R115: footprint sdi-mipi-cross-converter-footprints:0603-res -> sdi-mipi-video-converter-footprints:0603-res; symbol sdi-mipi-cross-converter:R_10k_0603 -> sdi-mipi-video-converter:R_10k_0603
- R107, R108, R118: footprint sdi-mipi-cross-converter-footprints:0603-res -> sdi-mipi-video-converter-footprints:0603-res; symbol sdi-mipi-cross-converter:R_15k_0603 -> sdi-mipi-video-converter:R_15k_0603
- R109, R110, R121, R122, R123, R124, R125, R126, R127, R128, R129, R130, R73, R74: footprint sdi-mipi-cross-converter-footprints:0402-res -> sdi-mipi-video-converter-footprints:0402-res; symbol sdi-mipi-cross-converter:R_0R_0402 -> sdi-mipi-video-converter:R_0R_0402
- R11, R8: footprint sdi-mipi-cross-converter-footprints:0402-res -> sdi-mipi-video-converter-footprints:0402-res; symbol sdi-mipi-cross-converter:R_5k1_0402 -> sdi-mipi-video-converter:R_5k1_0402
- R116, R117, R119: footprint sdi-mipi-cross-converter-footprints:0603-res -> sdi-mipi-video-converter-footprints:0603-res; symbol sdi-mipi-cross-converter:R_0R_0603 -> sdi-mipi-video-converter:R_0R_0603
- R133, R134: footprint sdi-mipi-cross-converter-footprints:0402-res -> sdi-mipi-video-converter-footprints:0402-res; symbol sdi-mipi-cross-converter:R_27R_0402 -> sdi-mipi-video-converter:R_27R_0402
- SW1: footprint sdi-mipi-cross-converter-footprints:SW_DIP_SPSTx02_Slide_Copal_CVS-02xB_W5.9mm_P1mm -> sdi-mipi-video-converter-footprints:SW_DIP_SPSTx02_Slide_Copal_CVS-02xB_W5.9mm_P1mm; symbol sdi-mipi-cross-converter:CVS-02B -> sdi-mipi-video-converter:CVS-02B
- TP44, TP45, TP46, TP47: footprint sdi-mipi-cross-converter-footprints:Testpoint_smd_0_75mm -> sdi-mipi-video-converter-footprints:Testpoint_smd_0_75mm; symbol sdi-mipi-cross-converter:TP_SMD_0_75MM -> sdi-mipi-video-converter:TP_SMD_0_75MM
- U11: footprint sdi-mipi-cross-converter-footprints:BGA-256_16x16_14.0x14.0mm -> sdi-mipi-video-converter-footprints:BGA-256_16x16_14.0x14.0mm; symbol sdi-mipi-cross-converter:LIFCL-40-9BG256C -> sdi-mipi-video-converter:LIFCL-40-9BG256C
- U13, U14, U19: footprint sdi-mipi-cross-converter-footprints:SOT23-6L -> sdi-mipi-video-converter-footprints:SOT23-6L; symbol sdi-mipi-cross-converter:DIO7553ST6 -> sdi-mipi-video-converter:DIO7553ST6
- U20: footprint sdi-mipi-cross-converter-footprints:WQFN-16-1EP_4x4mm -> sdi-mipi-video-converter-footprints:WQFN-16-1EP_4x4mm; symbol sdi-mipi-cross-converter:FT230XQ-R -> sdi-mipi-video-converter:FT230XQ-R
Other:
- title: SDI-MIPI Cross Converter -> SDI-MIPI Video Converter
