File: peripherals.kicad_sch (KiCad schematic)
At the start: 75 parts, among them J1 USB-C_USB4105-GF-A, J10 PinHeader_1x6_P2.54mm_SMD_Hor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, J4 Conn_FFC_WE_68715014522_ONE-S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, J5 PinHeader_2x5_P1.27mm_SMD, J6 Conn_FFC_WE_68715014522_ONE-S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, J8 SM04B-SRSS-TB-LF-SN, J9 JST_GH_1x6_SM06B-SRSS-TB-LF-SN, SW1 SW_CVS-02B, U11 LIFCL-40-9BG256C, U13 DIO7553ST6, U14 DIO7553ST6, U19 DIO7553ST6, U20 FT230X_QFN

Commit message: [#55653] Fix LIFCL-40
Parts:
- J10: footprint antmicro-footprints:PinHeader_1x6_P2.54mm_SMD_Horizontal -> sdi-mipi-video-converter-footprints:PinHeader_1x6_P2.54mm_SMD_Horizontal; symbol antmicroGenericPinHeaders:PinHeader_1x6_P2.54mm_SMD_Horizontal -> sdi-mipi-video-converter:PinHeader_1x6_P2.54mm_SMD_Horizontal
- J8: footprint antmicro-footprints:Conn_JST_SH_1x4_SM04B-SRSS-TB-LF-SN -> sdi-mipi-video-converter-footprints:Conn_JST_SH_1x4_SM04B-SRSS-TB-LF-SN; symbol antmicroWire2BoardConnectors:JST_SH_1x4_SM04B-SRSS-TB-LF-SN -> sdi-mipi-video-converter:JST_SH_1x4_SM04B-SRSS-TB-LF-SN
- J9: footprint antmicro-footprints:Conn_JST_GH_1x6_SM06B-SRSS-TB-LF-SN -> sdi-mipi-video-converter-footprints:Conn_JST_GH_1x6_SM06B-SRSS-TB-LF-SN; symbol antmicroWire2BoardConnectors:JST_GH_1x6_SM06B-SRSS-TB-LF-SN -> sdi-mipi-video-converter:JST_GH_1x6_SM06B-SRSS-TB-LF-SN
- U11: footprint antmicro-footprints:BGA-256_14x14mm_Layout16x16_P0.8x0.8mm_LATTICE -> sdi-mipi-video-converter-footprints:BGA-256_14x14mm_Layout16x16_P0.8x0.8mm_LATTICE
- U11: value LIFCL-40-9BG256C -> CrossLink_LIFCL-40-9BG256C; footprint antmicro-footprints:BGA-256_14x14mm_Layout16x16_P0.8x0.8mm_LATTICE -> sdi-mipi-video-converter-footprints:BGA-256_14x14mm_Layout16x16_P0.8x0.8mm_LATTICE; symbol sdi-mipi-video-converter:LIFCL-40-9BG256C -> sdi-mipi-video-converter:CrossLink_LIFCL-40-9BG256C; Manufacturer Lattice -> Lattice Semiconductor
- U20: footprint antmicro-footprints:QFN-16-1EP_4x4mm_P0.65mm -> sdi-mipi-video-converter-footprints:QFN-16-1EP_4x4mm_P0.65mm; symbol antmicroInterfaceControllers:FT230X_QFN -> sdi-mipi-video-converter:FT230X_QFN
Changed lines of the file:
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@@
     )
   )
-  (symbol (lib_id "antmicroWire2BoardConnectors:JST_GH_1x6_SM06B-SRSS-TB-LF-SN") (at 377.19 35.56 0) (unit 1)
+  (symbol (lib_id "sdi-mipi-video-converter:JST_GH_1x6_SM06B-SRSS-TB-LF-SN") (at 377.19 35.56 0) (unit 1)
     (in_bom yes) (on_board yes) (dnp no) (fields_autoplaced)
     (property "Reference" "J9" (at 384.81 43.18 0)
@@
       (effects (font (size 1.27 1.27) (thickness 0.15)) (justify left bottom) hide)
     )
-    (property "Footprint" "antmicro-footprints:Conn_JST_GH_1x6_SM06B-SRSS-TB-LF-SN" (at 403.86 45.72 0)
+    (property "Footprint" "sdi-mipi-video-converter-footprints:Conn_JST_GH_1x6_SM06B-SRSS-TB-LF-SN" (at 403.86 45.72 0)
       (effects (font (size 1.27 1.27) (thickness 0.15)) (justify left bottom) hide)
     )
@@
     )
   )
-  (symbol (lib_id "antmicroGenericPinHeaders:PinHeader_1x6_P2.54mm_SMD_Horizontal") (at 381 69.85 0) (unit 1)
+  (symbol (lib_id "sdi-mipi-video-converter:PinHeader_1x6_P2.54mm_SMD_Horizontal") (at 381 69.85 0) (unit 1)
     (in_bom yes) (on_board yes) (dnp no) (fields_autoplaced)
     (property "Reference" "J10" (at 387.35 73.66 0)
@@
       (effects (font (size 1.27 1.27) (thickness 0.15)) (justify left bottom) hide)
     )
-    (property "Footprint" "antmicro-footprints:PinHeader_1x6_P2.54mm_SMD_Horizontal" (at 400.05 81.28 0)
+    (property "Footprint" "sdi-mipi-video-converter-footprints:PinHeader_1x6_P2.54mm_SMD_Horizontal" (at 400.05 81.28 0)
       (effects (font (size 1.27 1.27) (thickness 0.15)) (justify left bottom) hide)
     )
@@
       (effects (font (size 1.27 1.27) (thickness 0.15)))
     )
-    (property "Footprint" "antmicro-footprints:BGA-256_14x14mm_Layout16x16_P0.8x0.8mm_LATTICE" (at 33.02 72.39 0)
+    (property "Footprint" "sdi-mipi-video-converter-footprints:BGA-256_14x14mm_Layout16x16_P0.8x0.8mm_LATTICE" (at 33.02 72.39 0)
       (effects (font (size 1.27 1.27) (thickness 0.15)) (justify left bottom) hide)
     )
@@
     )
   )
-  (symbol (lib_id "antmicroWire2BoardConnectors:JST_SH_1x4_SM04B-SRSS-TB-LF-SN") (at 43.815 200.66 0) (unit 1)
+  (symbol (lib_id "sdi-mipi-video-converter:JST_SH_1x4_SM04B-SRSS-TB-LF-SN") (at 43.815 200.66 0) (unit 1)
     (in_bom yes) (on_board yes) (dnp no)
     (property "Reference" "J8" (at 52.07 204.47 0)
@@
       (effects (font (size 1.27 1.27) (thickness 0.15)) (justify left) hide)
     )
-    (property "Footprint" "antmicro-footprints:Conn_JST_SH_1x4_SM04B-SRSS-TB-LF-SN" (at 70.485 210.82 0)
+    (property "Footprint" "sdi-mipi-video-converter-footprints:Conn_JST_SH_1x4_SM04B-SRSS-TB-LF-SN" (at 70.485 210.82 0)
       (effects (font (size 1.27 1.27) (thickness 0.15)) (justify left bottom) hide)
     )
@@
     )
   )
-  (symbol (lib_id "sdi-mipi-video-converter:LIFCL-40-9BG256C") (at 50.8 33.02 0) (mirror y) (unit 9)
+  (symbol (lib_id "sdi-mipi-video-converter:CrossLink_LIFCL-40-9BG256C") (at 50.8 33.02 0) (mirror y) (unit 9)
     (in_bom yes) (on_board yes) (dnp no) (fields_autoplaced)
     (property "Reference" "U11" (at 36.195 25.4 0)
       (effects (font (size 1.27 1.27) (thickness 0.15)))
     )
-    (property "Value" "LIFCL-40-9BG256C" (at 36.195 27.94 0)
-      (effects (font (size 1.27 1.27) (thickness 0.15)))
-    )
-    (property "Footprint" "antmicro-footprints:BGA-256_14x14mm_Layout16x16_P0.8x0.8mm_LATTICE" (at -8.89 25.4 0)
+    (property "Value" "CrossLink_LIFCL-40-9BG256C" (at -2.54 38.1 0)
       (effects (font (size 1.27 1.27) (thickness 0.15)) (justify left bottom) hide)
     )
-    (property "Datasheet" "https://www.latticesemi.com/-/media/LatticeSemi/Documents/DataSheets/CrossLink/FPGA-DS-02007-2-1-CrossLink-Family-Data-Sheet.ashx?document_id=51662" (at -8.89 27.94 0)
+    (property "Footprint" "sdi-mipi-video-converter-footprints:BGA-256_14x14mm_Layout16x16_P0.8x0.8mm_LATTICE" (at -2.54 40.64 0)
       (effects (font (size 1.27 1.27) (thickness 0.15)) (justify left bottom) hide)
     )
-    (property "MPN" "LIFCL-40-9BG256C" (at -8.89 30.48 0)
+    (property "Datasheet" "https://www.latticesemi.com/-/media/LatticeSemi/Documents/DataSheets/CrossLink/FPGA-DS-02007-2-1-CrossLink-Family-Data-Sheet.ashx?document_id=51662" (at -2.54 43.18 0)
       (effects (font (size 1.27 1.27) (thickness 0.15)) (justify left bottom) hide)
     )
-    (property "Manufacturer" "Lattice" (at -8.89 33.02 0)
+    (property "MPN" "LIFCL-40-9BG256C" (at 36.195 27.94 0)
+      (effects (font (size 1.27 1.27) (thickness 0.15)))
+    )
+    (property "Manufacturer" "Lattice Semiconductor" (at -2.54 45.72 0)
       (effects (font (size 1.27 1.27) (thickness 0.15)) (justify left bottom) hide)
     )
-    (property "Author" "Antmicro" (at -8.89 35.56 0)
+    (property "Author" "Antmicro" (at -2.54 48.26 0)
       (effects (font (size 1.27 1.27) (thickness 0.15)) (justify left bottom) hide)
     )
-    (property "License" "Apache-2.0" (at -8.89 38.1 0)
+    (property "License" "Apache-2.0" (at -2.54 50.8 0)
       (effects (font (size 1.27 1.27) (thickness 0.15)) (justify left bottom) hide)
     )
@@
       (effects (font (size 1.27 1.27) (thickness 0.15)))
     )
-    (property "Footprint" "antmicro-footprints:BGA-256_14x14mm_Layout16x16_P0.8x0.8mm_LATTICE" (at 45.72 25.4 0)
+    (property "Footprint" "sdi-mipi-video-converter-footprints:BGA-256_14x14mm_Layout16x16_P0.8x0.8mm_LATTICE" (at 45.72 25.4 0)
       (effects (font (size 1.27 1.27) (thickness 0.15)) (justify left bottom) hide)
     )
@@
     )
   )
-  (symbol (lib_id "antmicroInterfaceControllers:FT230X_QFN") (at 314.96 217.17 0) (unit 1)
+  (symbol (lib_id "sdi-mipi-video-converter:FT230X_QFN") (at 314.96 217.17 0) (unit 1)
     (in_bom yes) (on_board yes) (dnp no) (fields_autoplaced)
     (property "Reference" "U20" (at 326.39 209.55 0)
@@
       (effects (font (size 1.27 1.27) (thickness 0.15)))
     )
-    (property "Footprint" "antmicro-footprints:QFN-16-1EP_4x4mm_P0.65mm" (at 354.33 229.87 0)
+    (property "Footprint" "sdi-mipi-video-converter-footprints:QFN-16-1EP_4x4mm_P0.65mm" (at 354.33 229.87 0)
       (effects (font (size 1.27 1.27) (thickness 0.15)) (justify left bottom) hide)
     )
@@
       (effects (font (size 1.27 1.27) (thickness 0.15)))
     )
-    (property "Footprint" "antmicro-footprints:BGA-256_14x14mm_Layout16x16_P0.8x0.8mm_LATTICE" (at 19.05 118.11 0)
+    (property "Footprint" "sdi-mipi-video-converter-footprints:BGA-256_14x14mm_Layout16x16_P0.8x0.8mm_LATTICE" (at 19.05 118.11 0)
       (effects (font (size 1.27 1.27) (thickness 0.15)) (justify left bottom) hide)
     )

Commit message: [#55653] Fix manufacturer of LIFCL-40
Parts:
- U11: footprint sdi-mipi-video-converter-footprints:BGA-256_14x14mm_Layout16x16_P0.8x0.8mm_LATTICE -> antmicro-footprints:BGA-256_14x14mm_Layout16x16_P0.8x0.8mm_LATTICE; symbol sdi-mipi-video-converter:LIFCL-40-9BG256C -> antmicroFPGAChips:CrossLink_LIFCL-40-9BG256C; Manufacturer Lattice -> Lattice Semiconductor
- U11: value CrossLink_LIFCL-40-9BG256C -> LIFCL-40-9BG256C; footprint sdi-mipi-video-converter-footprints:BGA-256_14x14mm_Layout16x16_P0.8x0.8mm_LATTICE -> antmicro-footprints:BGA-256_14x14mm_Layout16x16_P0.8x0.8mm_LATTICE; symbol sdi-mipi-video-converter:CrossLink_LIFCL-40-9BG256C -> antmicroFPGAChips:CrossLink_LIFCL-40-9BG256C
Changed lines of the file:
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@@
     )
   )
-  (symbol (lib_id "sdi-mipi-video-converter:LIFCL-40-9BG256C") (at 92.71 80.01 0) (mirror y) (unit 6)
+  (symbol (lib_id "antmicroFPGAChips:CrossLink_LIFCL-40-9BG256C") (at 92.71 80.01 0) (mirror y) (unit 6)
     (in_bom yes) (on_board yes) (dnp no) (fields_autoplaced)
     (property "Reference" "U11" (at 64.77 72.39 0)
       (effects (font (size 1.27 1.27) (thickness 0.15)))
     )
-    (property "Value" "LIFCL-40-9BG256C" (at 64.77 74.93 0)
-      (effects (font (size 1.27 1.27) (thickness 0.15)))
-    )
-    (property "Footprint" "sdi-mipi-video-converter-footprints:BGA-256_14x14mm_Layout16x16_P0.8x0.8mm_LATTICE" (at 33.02 72.39 0)
-      (effects (font (size 1.27 1.27) (thickness 0.15)) (justify left bottom) hide)
-    )
-    (property "Datasheet" "https://www.latticesemi.com/-/media/LatticeSemi/Documents/DataSheets/CrossLink/FPGA-DS-02007-2-1-CrossLink-Family-Data-Sheet.ashx?document_id=51662" (at 33.02 74.93 0)
-      (effects (font (size 1.27 1.27) (thickness 0.15)) (justify left bottom) hide)
-    )
-    (property "MPN" "LIFCL-40-9BG256C" (at 33.02 77.47 0)
-      (effects (font (size 1.27 1.27) (thickness 0.15)) (justify left bottom) hide)
-    )
-    (property "Manufacturer" "Lattice" (at 33.02 80.01 0)
-      (effects (font (size 1.27 1.27) (thickness 0.15)) (justify left bottom) hide)
-    )
-    (property "Author" "Antmicro" (at 33.02 82.55 0)
-      (effects (font (size 1.27 1.27) (thickness 0.15)) (justify left bottom) hide)
-    )
-    (property "License" "Apache-2.0" (at 33.02 85.09 0)
+    (property "Value" "LIFCL-40-9BG256C" (at 64.77 72.39 0)
+      (effects (font (size 1.27 1.27) (thickness 0.15)) hide)
+    )
+    (property "Footprint" "antmicro-footprints:BGA-256_14x14mm_Layout16x16_P0.8x0.8mm_LATTICE" (at 39.37 87.63 0)
+      (effects (font (size 1.27 1.27) (thickness 0.15)) (justify left bottom) hide)
+    )
+    (property "Datasheet" "https://www.latticesemi.com/-/media/LatticeSemi/Documents/DataSheets/CrossLink/FPGA-DS-02007-2-1-CrossLink-Family-Data-Sheet.ashx?document_id=51662" (at 39.37 90.17 0)
+      (effects (font (size 1.27 1.27) (thickness 0.15)) (justify left bottom) hide)
+    )
+    (property "MPN" "LIFCL-40-9BG256C" (at 64.77 74.93 0)
+      (effects (font (size 1.27 1.27) (thickness 0.15)))
+    )
+    (property "Manufacturer" "Lattice Semiconductor" (at 39.37 92.71 0)
+      (effects (font (size 1.27 1.27) (thickness 0.15)) (justify left bottom) hide)
+    )
+    (property "Author" "Antmicro" (at 39.37 95.25 0)
+      (effects (font (size 1.27 1.27) (thickness 0.15)) (justify left bottom) hide)
+    )
+    (property "License" "Apache-2.0" (at 39.37 97.79 0)
       (effects (font (size 1.27 1.27) (thickness 0.15)) (justify left bottom) hide)
     )
@@
     )
   )
-  (symbol (lib_id "sdi-mipi-video-converter:CrossLink_LIFCL-40-9BG256C") (at 50.8 33.02 0) (mirror y) (unit 9)
+  (symbol (lib_id "antmicroFPGAChips:CrossLink_LIFCL-40-9BG256C") (at 50.8 33.02 0) (mirror y) (unit 9)
     (in_bom yes) (on_board yes) (dnp no) (fields_autoplaced)
     (property "Reference" "U11" (at 36.195 25.4 0)
       (effects (font (size 1.27 1.27) (thickness 0.15)))
     )
-    (property "Value" "CrossLink_LIFCL-40-9BG256C" (at -2.54 38.1 0)
-      (effects (font (size 1.27 1.27) (thickness 0.15)) (justify left bottom) hide)
-    )
-    (property "Footprint" "sdi-mipi-video-converter-footprints:BGA-256_14x14mm_Layout16x16_P0.8x0.8mm_LATTICE" (at -2.54 40.64 0)
+    (property "Value" "LIFCL-40-9BG256C" (at -2.54 38.1 0)
+      (effects (font (size 1.27 1.27) (thickness 0.15)) (justify left bottom) hide)
+    )
+    (property "Footprint" "antmicro-footprints:BGA-256_14x14mm_Layout16x16_P0.8x0.8mm_LATTICE" (at -2.54 40.64 0)
       (effects (font (size 1.27 1.27) (thickness 0.15)) (justify left bottom) hide)
     )
@@
     )
   )
-  (symbol (lib_id "sdi-mipi-video-converter:LIFCL-40-9BG256C") (at 105.41 33.02 0) (mirror y) (unit 10)
+  (symbol (lib_id "antmicroFPGAChips:CrossLink_LIFCL-40-9BG256C") (at 105.41 33.02 0) (mirror y) (unit 10)
     (in_bom yes) (on_board yes) (dnp no) (fields_autoplaced)
     (property "Reference" "U11" (at 90.805 25.4 0)
       (effects (font (size 1.27 1.27) (thickness 0.15)))
     )
-    (property "Value" "LIFCL-40-9BG256C" (at 90.805 27.94 0)
-      (effects (font (size 1.27 1.27) (thickness 0.15)))
-    )
-    (property "Footprint" "sdi-mipi-video-converter-footprints:BGA-256_14x14mm_Layout16x16_P0.8x0.8mm_LATTICE" (at 45.72 25.4 0)
-      (effects (font (size 1.27 1.27) (thickness 0.15)) (justify left bottom) hide)
-    )
-    (property "Datasheet" "https://www.latticesemi.com/-/media/LatticeSemi/Documents/DataSheets/CrossLink/FPGA-DS-02007-2-1-CrossLink-Family-Data-Sheet.ashx?document_id=51662" (at 45.72 27.94 0)
-      (effects (font (size 1.27 1.27) (thickness 0.15)) (justify left bottom) hide)
-    )
-    (property "MPN" "LIFCL-40-9BG256C" (at 45.72 30.48 0)
-      (effects (font (size 1.27 1.27) (thickness 0.15)) (justify left bottom) hide)
-    )
-    (property "Manufacturer" "Lattice" (at 45.72 33.02 0)
-      (effects (font (size 1.27 1.27) (thickness 0.15)) (justify left bottom) hide)
-    )
-    (property "Author" "Antmicro" (at 45.72 35.56 0)
-      (effects (font (size 1.27 1.27) (thickness 0.15)) (justify left bottom) hide)
-    )
-    (property "License" "Apache-2.0" (at 45.72 38.1 0)
+    (property "Value" "LIFCL-40-9BG256C" (at 90.805 25.4 0)
+      (effects (font (size 1.27 1.27) (thickness 0.15)) hide)
+    )
+    (property "Footprint" "antmicro-footprints:BGA-256_14x14mm_Layout16x16_P0.8x0.8mm_LATTICE" (at 52.07 40.64 0)
+      (effects (font (size 1.27 1.27) (thickness 0.15)) (justify left bottom) hide)
+    )
+    (property "Datasheet" "https://www.latticesemi.com/-/media/LatticeSemi/Documents/DataSheets/CrossLink/FPGA-DS-02007-2-1-CrossLink-Family-Data-Sheet.ashx?document_id=51662" (at 52.07 43.18 0)
+      (effects (font (size 1.27 1.27) (thickness 0.15)) (justify left bottom) hide)
+    )
+    (property "MPN" "LIFCL-40-9BG256C" (at 90.805 27.94 0)
+      (effects (font (size 1.27 1.27) (thickness 0.15)))
+    )
+    (property "Manufacturer" "Lattice Semiconductor" (at 52.07 45.72 0)
+      (effects (font (size 1.27 1.27) (thickness 0.15)) (justify left bottom) hide)
+    )
+    (property "Author" "Antmicro" (at 52.07 48.26 0)
+      (effects (font (size 1.27 1.27) (thickness 0.15)) (justify left bottom) hide)
+    )
+    (property "License" "Apache-2.0" (at 52.07 50.8 0)
       (effects (font (size 1.27 1.27) (thickness 0.15)) (justify left bottom) hide)
     )
@@
     )
   )
-  (symbol (lib_id "sdi-mipi-video-converter:LIFCL-40-9BG256C") (at 78.74 125.73 0) (mirror y) (unit 2)
+  (symbol (lib_id "antmicroFPGAChips:CrossLink_LIFCL-40-9BG256C") (at 78.74 125.73 0) (mirror y) (unit 2)
     (in_bom yes) (on_board yes) (dnp no) (fields_autoplaced)
     (property "Reference" "U11" (at 55.88 118.11 0)
       (effects (font (size 1.27 1.27) (thickness 0.15)))
     )
-    (property "Value" "LIFCL-40-9BG256C" (at 55.88 120.65 0)
-      (effects (font (size 1.27 1.27) (thickness 0.15)))
-    )
-    (property "Footprint" "sdi-mipi-video-converter-footprints:BGA-256_14x14mm_Layout16x16_P0.8x0.8mm_LATTICE" (at 19.05 118.11 0)
-      (effects (font (size 1.27 1.27) (thickness 0.15)) (justify left bottom) hide)
-    )
-    (property "Datasheet" "https://www.latticesemi.com/-/media/LatticeSemi/Documents/DataSheets/CrossLink/FPGA-DS-02007-2-1-CrossLink-Family-Data-Sheet.ashx?document_id=51662" (at 19.05 120.65 0)
-      (effects (font (size 1.27 1.27) (thickness 0.15)) (justify left bottom) hide)
-    )
-    (property "MPN" "LIFCL-40-9BG256C" (at 19.05 123.19 0)
-      (effects (font (size 1.27 1.27) (thickness 0.15)) (justify left bottom) hide)
-    )
-    (property "Manufacturer" "Lattice" (at 19.05 125.73 0)
-      (effects (font (size 1.27 1.27) (thickness 0.15)) (justify left bottom) hide)
-    )
-    (property "Author" "Antmicro" (at 19.05 128.27 0)
-      (effects (font (size 1.27 1.27) (thickness 0.15)) (justify left bottom) hide)
-    )
-    (property "License" "Apache-2.0" (at 19.05 130.81 0)
-      (effects (font (size 1.27 1.27) (thickness 0.15)) (justify left bottom) hide)
-    )
+    (property "Value" "LIFCL-40-9BG256C" (at 55.88 118.11 0)
+      (effects (font (size 1.27 1.27) (thickness 0.15)) hide)
+    )
+    (property "Footprint" "antmicro-footprints:BGA-256_14x14mm_Layout16x16_P0.8x0.8mm_LATTICE" (at 25.4 133.35 0)
+      (effects (font (size 1.27 1.27) (thickness 0.15)) (justify left bottom) hide)
+    )
+    (property "Datasheet" "https://www.latticesemi.com/-/media/LatticeSemi/Documents/DataSheets/CrossLink/FPGA-DS-02007-2-1-CrossLink-Family-Data-Sheet.ashx?document_id=51662" (at 25.4 135.89 0)
+      (effects (font (size 1.27 1.27) (thickness 0.15)) (justify left bottom) hide)
+    )
+    (property "MPN" "LIFCL-40-9BG256C" (at 55.88 120.65 0)
+      (effects (font (size 1.27 1.27) (thickness 0.15)))
+    )
+    (property "Manufacturer" "Lattice Semiconductor" (at 25.4 138.43 0)
+      (effects (font (size 1.27 1.27) (thickness 0.15)) (justify left bottom) hide)
+    )
+    (property "Author" "Antmicro" (at 25.4 140.97 0)
+      (effects (font (size 1.27 1.27) (thickness 0.15)) (justify left bottom) hide)
+    )
+    (property "License" "Apache-2.0" (at 25.4 143.51 0)
+      (effects (font (size 1.27 1.27) (thickness 0.15)) (justify left bottom) hide)
+    )
