File: FPGA_Power.kicad_sch (KiCad schematic)
At the start: 31 parts, among them U11 LIFCL-40-9BG256C

Commit message: [#48149] Change LIFCL footprint for footprint with markings
Parts:
- U11: footprint sdi-mipi-video-converter-footprints:BGA-256_14x14mm_Layout16x16_P0.8x0.8mm -> antmicro-footprints:BGA-256_14x14mm_Layout16x16_P0.8x0.8mm_LATTICE
Changed lines of the file:
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@@
       (effects (font (size 1.27 1.27) (thickness 0.15)))
     )
-    (property "Footprint" "sdi-mipi-video-converter-footprints:BGA-256_14x14mm_Layout16x16_P0.8x0.8mm" (id 2) (at 314.96 109.22 0)
+    (property "Footprint" "antmicro-footprints:BGA-256_14x14mm_Layout16x16_P0.8x0.8mm_LATTICE" (id 2) (at 314.96 109.22 0)
       (effects (font (size 1.27 1.27) (thickness 0.15)) (justify left bottom) hide)
     )

Commit message: [#48149] Update GS297 and LIFCL symbols, update local lib
Parts:
- U11: footprint antmicro-footprints:BGA-256_14x14mm_Layout16x16_P0.8x0.8mm_LATTICE -> sdi-mipi-video-converter-footprints:BGA-256_14x14mm_Layout16x16_P0.8x0.8mm_LATTICE

Commit message: Update SCH and PCB revision date
Parts:
- U11: footprint sdi-mipi-video-converter-footprints:BGA-256_14x14mm_Layout16x16_P0.8x0.8mm_LATTICE -> antmicro-footprints:BGA-256_14x14mm_Layout16x16_P0.8x0.8mm_LATTICE
