File: sdi-mipi-video-converter.kicad_sch (KiCad schematic)
At the start: 0 parts

Commit message: [#82595] Project refresh 81589
Parts:
- added MP1, MP2, MP3, MP4: MP_Pad5.4mm_Drill2.7mm, antmicro-footprints:MP_Pad5.4mm_Drill2.7mm, symbol antmicroMechanicalParts:MP_Pad5.4mm_Drill2.7mm
Connections:
- no-connect marks 0 -> 4
